File: PCB/leanometer_esp32/leanometer_esp32.kicad_pcb (KiCad board)
At the start: 4 copper layers, 70 parts, among them J1 Conn_01x07, J2 PROG, J3 VBAT, J4 DM3AT-SF-PEJM5, J5 MPU6050, J6 Conn_01x07, Q1 BSS138, SW1 SW_Push, SW2 SW_Push, SW3 SW_Push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

Commit message: Added PowerBoard hierarchical sheet, completed layout
Signed-off-by: theloukou
Parts:
- removed FID1, FID2, FID3: Fiducial, Fiducial:Fiducial_0.75mm_Mask1.5mm
- added J7: Conn_01x03, Connector_PinHeader_2.54mm:PinHeader_1x03_P2.54mm_Vertical, F.Cu at (97.0, 116.8)
- added U8: GY-521, MPU6050(GY-521):GY-521_NoSlave+AD0, F.Cu at (96.5, 86.1)
- C1: moved to F.Cu
- J5: value MPU6050 -> Conn_01x03; footprint Connector_PinHeader_2.54mm:PinHeader_1x04_P2.54mm_Vertical -> Connector_PinHeader_2.54mm:PinHeader_1x03_P2.54mm_Vertical
- moved C14 136.2 mm to (149.2, 92.9)
- moved C15 136.2 mm to (149.2, 106.6)
- moved U4 136.2 mm to (145.4, 101.5)
- moved U5 136.2 mm to (145.4, 87.8)
- moved U6 136.2 mm to (137.8, 106.6)
- moved U7 136.2 mm to (137.8, 92.9)
- moved J6 136.2 mm to (132.0, 90.6)
- moved R15 136.2 mm to (132.5, 82.8)
- moved R16 136.2 mm to (132.5, 84.5)
- moved R18 136.2 mm to (149.5, 96.4)
- moved R19 136.2 mm to (141.4, 99.0)
- moved R20 136.2 mm to (141.4, 104.0)
- moved R21 136.2 mm to (141.4, 106.6)
- moved R23 136.2 mm to (149.5, 106.6)
- moved R24 136.2 mm to (141.4, 96.4)
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Connections:
- J1 pad 2: /DisplayBoard/DISP_DATA -> /DisplayBoard/DISP_BRIGHT
- J1 pad 3: /DisplayBoard/DISP_CLOCK -> /DisplayBoard/DISP_LATCH
- J1 pad 4: /DisplayBoard/DISP_LATCH -> /DisplayBoard/DISP_CLOCK
- J1 pad 5: /DisplayBoard/DISP_BRIGHT -> /DisplayBoard/DISP_DATA
- J2 pad 1: +BATT -> +3V3
- J5 pad 3: /MainBoard/I2C_SCL -> /MainBoard/ADC_VBAT
- J6 pad 2: /DisplayBoard/DISP_DATA -> /DisplayBoard/DISP_BRIGHT
- J6 pad 3: /DisplayBoard/DISP_CLOCK -> /DisplayBoard/DISP_LATCH
- J6 pad 4: /DisplayBoard/DISP_LATCH -> /DisplayBoard/DISP_CLOCK
- J6 pad 5: /DisplayBoard/DISP_BRIGHT -> /DisplayBoard/DISP_DATA
- U2 pad 27: /MainBoard/BUT -> unconnected-(U2-IO16-Pad27)
Routing:
- net /DisplayBoard/DISP_CLOCK: track 0.00 -> 92.2 mm, vias 0 -> 1
- net /DisplayBoard/DISP_LATCH: track 0.00 -> 91.5 mm, vias 0 -> 2
- net /DisplayBoard/DISP_DATA: track 0.00 -> 78.7 mm, vias 0 -> 2
- net +3V3: track 0.00 -> 77.9 mm, vias 0 -> 18
- net /DisplayBoard/ADC_LDR: track 0.00 -> 67.8 mm, vias 0 -> 1
- net /MainBoard/SD_MOSI: track 0.00 -> 61.6 mm, vias 0 -> 2
- net /DisplayBoard/DISP_BRIGHT: track 0.00 -> 61.3 mm, vias 0 -> 2
- net /MainBoard/SD_SS: track 0.00 -> 50.6 mm, vias 0 -> 2
- net /DisplayBoard/LED_CATH: track 0.00 -> 48.4 mm, vias 0 -> 3
- net /MainBoard/SD_DET_B: track 0.00 -> 47.3 mm
- net /MainBoard/SD_MISO: track 0.00 -> 43.6 mm, vias 0 -> 2
- net /MainBoard/I2C_SCL: track 0.00 -> 42.7 mm, vias 0 -> 2
- net /MainBoard/SD_SCK: track 0.00 -> 40.9 mm, vias 0 -> 2
- net GND: track 0.00 -> 40.2 mm, vias 0 -> 32
- net /MainBoard/IMU_INT: track 0.00 -> 35.8 mm, vias 0 -> 4
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- added copper zone on In2.Cu, net +3V3
- added copper zone on B.Cu, net GND
- added copper zone on F.Cu, net GND
- added copper zone on In1.Cu, net GND
Other:
- board outline added: 95.5 x 58.5 mm

Commit message: Full layout rework
Signed-off-by: theloukou
Parts:
- C1: moved to B.Cu
- moved C5 86.7 mm to (155.0, 117.0), turned to 90 degrees
- moved C6 84.7 mm to (152.7, 117.0), turned to -90 degrees
- moved R4 82.7 mm to (155.0, 113.2), turned to 90 degrees
- moved C3 80.5 mm to (152.7, 113.2), turned to 90 degrees
- moved R5 77.6 mm to (156.3, 109.3)
- moved SW2 77.6 mm to (156.3, 108.6)
- moved C4 67.2 mm to (119.0, 67.0), turned to 0 degrees
- moved U2 66.3 mm to (140.6, 109.4), turned to 180 degrees
- moved D1 64.7 mm to (106.6, 65.5), turned to 0 degrees
- moved C2 63.8 mm to (113.9, 67.0), turned to 0 degrees
- moved J2 60.5 mm to (121.7, 111.0)
- moved C1 58.5 mm to (146.8, 108.1)
- moved U1 56.3 mm to (116.4, 71.8), turned to 0 degrees
- moved R8 49.3 mm to (139.7, 94.9), turned to 180 degrees
- moved J3 48.6 mm to (109.5, 73.8), turned to 90 degrees
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Connections:
- U2 pad 27: unconnected-(U2-IO16-Pad27) -> /MainBoard/BUT
Routing:
- net /DisplayBoard/ADC_LDR: track 67.8 -> 31.4 mm
- net /DisplayBoard/DISP_DATA: track 78.7 -> 42.7 mm, vias 2 -> 1
- net /DisplayBoard/DISP_CLOCK: track 92.2 -> 56.6 mm, vias 1 -> 0
- net /DisplayBoard/DISP_LATCH: track 91.5 -> 58.3 mm, vias 2 -> 1
- net /MainBoard/ADC_VBAT: track 35.1 -> 64.7 mm, vias 0 -> 1
- net /MainBoard/SD_MOSI: track 61.6 -> 33.1 mm
- net /MainBoard/SD_SS: track 50.6 -> 25.9 mm, vias 2 -> 0
- net /DisplayBoard/DISP_BRIGHT: track 61.3 -> 37.8 mm, vias 2 -> 1
- net /MainBoard/BUT: track 7.54 -> 29.8 mm, vias 1 -> 3
- net /MainBoard/SD_SCK: track 40.9 -> 24.6 mm, vias 2 -> 0
- net /MainBoard/SD_DET_B: track 47.3 -> 33.4 mm, vias 0 -> 2
- net /MainBoard/SD_MISO: track 43.6 -> 31.9 mm, vias 2 -> 0
- net /MainBoard/I2C_SCL: track 42.7 -> 31.2 mm, vias 2 -> 1
- net /MainBoard/I2C_SDA: track 33.9 -> 24.8 mm, vias 2 -> 0
- net /MainBoard/IO0: track 12.2 -> 17.6 mm
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Other:
- board size 95.5 x 58.5 mm -> 91.3 x 63.8 mm

Commit message: Finalized PCB layout Added various texts Added BOM
Signed-off-by: theloukou
Parts:
- added C16: 100nF, Capacitor_SMD:C_0603_1608Metric, B.Cu at (152.4, 108.0)
Routing:
- net GND: vias 28 -> 29
Other:
- board text added: "+"
- board text added: "3V3"
- board text added: "3V3 GND TX RX"
- board text added: "BTN"
- board text added: "DisplayBoard R1"
- board text added: "EN"
- board text added: "ESP32 Leanometer R1 Lefteris Kantakos 2023 github.com/theloukou"
- board text added: "GND"
- board text added: "IO0"
- board text added: "PwrBoard R1"
- board text added: "VIN"

Commit message: Removed a million breakaway vias for proper cutouts Cleaned up track stubs
Signed-off-by: theloukou
Routing:
- net /MainBoard/I2C_SDA: track 24.8 -> 24.2 mm
- net (no net): vias 37 -> 0
Other:
- outline, holes or cut-outs redrawn
